Commit message: Restructure: rename dog_sim→dog_task, consolidate assets, adopt ik as subpackage
- Rename dog_sim/ → dog_task/ (python -m dog_task)
- Consolidate all static assets under assets/: go2/, d1/, rl_models/
- Move D1 IK solver into dog_task/modules/arm/ik/ as proper subpackage
  (replaces sys.path.insert hack with relative import)
- Remove ROS cruft from D1 URDF (CMakeLists.txt, launch/, package.xml)
- Remove duplicate STL files, fix URDF mesh paths
- Remove hardware/ and urdf/ top-level dirs
- Add .vscode/ to .gitignore
- Update all config paths and script references

Co-Authored-By: Claude Opus 4.7 <noreply@anthropic.com>

File: assets/d1/d1.urdf (robot description, URDF)
Before this commit: robot d1_550_description, 9 links, 8 joints
Links:
- link Empty_Link1: geometry collision mesh filename=meshes/Empty_Link1.STL; visual mesh filename=meshes/Empty_Link1.STL
- link Empty_Link2: geometry collision mesh filename=meshes/Empty_Link2.STL; visual mesh filename=meshes/Empty_Link2.STL
- link Empty_Link3: geometry collision mesh filename=meshes/Empty_Link3.STL; visual mesh filename=meshes/Empty_Link3.STL
- link Empty_Link4: geometry collision mesh filename=meshes/Empty_Link4.STL; visual mesh filename=meshes/Empty_Link4.STL
- link Empty_Link5: geometry collision mesh filename=meshes/Empty_Link5.STL; visual mesh filename=meshes/Empty_Link5.STL
- link Empty_Link6: geometry collision mesh filename=meshes/Empty_Link6.STL; visual mesh filename=meshes/Empty_Link6.STL
- link Empty_Link_L: geometry collision mesh filename=meshes/Empty_Link_L.STL; visual mesh filename=meshes/Empty_Link_L.STL
- link Empty_Link_R: geometry collision mesh filename=meshes/Empty_Link_R.STL; visual mesh filename=meshes/Empty_Link_R.STL
- link base_link: geometry collision mesh filename=meshes/base_link.STL; visual mesh filename=meshes/base_link.STL
